Commit message: scaled the model down and added simple collision

File: ingenious_ws/src/akatsuki_description/urdf/bot.xacro (robot description, xacro)
@@ -7,5 +7,5 @@
     <inertial>
       <origin
-   xyz="0 0.0 0.12"
+   xyz="0 0.0 0"
         rpy="0 0 3.142" />
       <mass
@@ -29,8 +29,9 @@
     <collision>
     <origin
-        xyz="0 0.0 0.12"
-        rpy="0 0 0" />
-      <geometry>
-     <box size="0.585 0.30 0.25"/>
+        xyz="0 0.0 0"
+        rpy="0 0 0" />
+      <geometry>
+     <mesh
+          filename="package://akatsuki_description/meshes/stl/only_chassis.stl" />
       </geometry>
     </collision>
@@ -86,5 +87,5 @@
     <inertial>
       <origin
-        xyz="0 0 0"
+        xyz="0 0 0.12"
         rpy="0 0 0" />
       <mass
@@ -98,19 +99,18 @@
       <geometry>
         <mesh
-          filename="package://akatsuki_description/meshes/stl/wheel.stl" scale="0.1 0.1 0.1"/>
-      </geometry>
-      <material
-        name="">
-        <color
-          rgba="0.79216 0.81961 0.93333 1" />
-      </material>
-    </visual>
-    <collision>
-      <origin
-         xyz="0 0.025 0"
-        rpy="0 0 0" />
-      <geometry>
-          <mesh
-          filename="package://akatsuki_description/meshes/stl/wheel.stl" scale="0.1 0.1 0.1"/>
+          filename="package://akatsuki_description/meshes/stl/wheel_left.stl" />
+      </geometry>
+      <material
+        name="">
+        <color
+          rgba="0.79216 0.81961 0.93333 1" />
+      </material>
+    </visual>
+    <collision>
+      <origin
+         xyz="0.05 0 0"
+        rpy="0 1.5707 0" />
+      <geometry>
+          <cylinder length="0.1" radius="0.12"/>
       </geometry>
     </collision>
@@ -120,5 +120,5 @@
     type="continuous">
     <origin
-      xyz="0.8 -0.8 0.04"
+      xyz="0.27 -0.3 0"
       rpy="0 0 0" />
     <parent
@@ -146,19 +146,18 @@
       <geometry>
         <mesh
-          filename="package://akatsuki_description/meshes/stl/wheel.stl" scale="0.1 0.1 0.1"/>
-      </geometry>
-      <material
-        name="">
-        <color
-          rgba="0.79216 0.81961 0.93333 1" />
-      </material>
-    </visual>
-    <collision>
-      <origin
-         xyz="0 0.025 0"
-        rpy="0 0 0" />
-      <geometry>
-         <mesh
-          filename="package://akatsuki_description/meshes/stl/wheel.stl" scale="0.1 0.1 0.1"/>
+          filename="package://akatsuki_description/meshes/stl/wheel_left.stl" />
+      </geometry>
+      <material
+        name="">
+        <color
+          rgba="0.79216 0.81961 0.93333 1" />
+      </material>
+    </visual>
+    <collision>
+      <origin
+         xyz="0.05 0 0"
+        rpy="0 1.5707 0" />
+      <geometry>
+         <cylinder length="0.1" radius="0.12"/>
       </geometry>
     </collision>
@@ -168,5 +167,5 @@
     type="continuous">
     <origin
-      xyz="0.8 0.8 0.04"
+      xyz="0.27 0.3 0"
       rpy="0 0 0" />
     <parent
@@ -194,5 +193,5 @@
       <geometry>
         <mesh
-          filename="package://akatsuki_description/meshes/stl/wheel.stl" scale="0.1 0.1 0.1"/>
+          filename="package://akatsuki_description/meshes/stl/wheel_right.stl" />
       </geometry>
       <material
@@ -204,9 +203,8 @@
    <collision>
       <origin
-         xyz="0 0.025 0"
-        rpy="0 0 0" />
-      <geometry>
-          <mesh
-          filename="package://akatsuki_description/meshes/stl/wheel.stl" scale="0.1 0.1 0.1"/>
+         xyz="-0.05 0 0"
+        rpy="0 1.5707 0" />
+      <geometry>
+          <cylinder length="0.1" radius="0.12"/>
       </geometry>
     </collision>
@@ -216,5 +214,5 @@
     type="continuous">
     <origin
-      xyz="-0.8 -0.8 0.04"
+      xyz="-0.27 -0.3 0"
       rpy="0 0 0" />
     <parent
@@ -242,5 +240,5 @@
       <geometry>
         <mesh
-          filename="package://akatsuki_description/meshes/stl/wheel.stl" scale="0.1 0.1 0.1"/>
+          filename="package://akatsuki_description/meshes/stl/wheel_right.stl" />
       </geometry>
       <material
@@ -252,9 +250,8 @@
    <collision>
       <origin
-         xyz="0 0.025 0"
-        rpy="0 0 0" />
-      <geometry>
-          <mesh
-          filename="package://akatsuki_description/meshes/stl/wheel.stl" scale="0.1 0.1 0.1"/>
+         xyz="-0.05 0 0"
+        rpy="0 1.5707 0" />
+      <geometry>
+          <cylinder length="0.1" radius="0.12"/>
       </geometry>
     </collision>
@@ -264,5 +261,5 @@
     type="continuous">
     <origin
-      xyz="-0.8 0.8 0.04"
+      xyz="-0.27 0.3 0"
       rpy="0 0 0" />
     <parent
@@ -275,5 +272,5 @@
 <joint name="bot_cam_joint" type="fixed">
     <axis xyz="0 0 0" />
-    <origin xyz="0 -1.05 0.1" rpy="0 0 0"/>
+    <origin xyz="0 -0.47 0.06" rpy="0 0 0"/>
     <parent link="obito_base"/>
     <child link="camera_link"/>
@@ -333,5 +330,5 @@
   <joint name="lidar_joint" type="fixed">
     <axis xyz="0 1 0"/>
-    <origin xyz="0 -0.9 0.5"
+    <origin xyz="0 -0.36 0.23"
       rpy="0 0 -1.571" />
     <parent link="obito_base"/>
