Commit message: updated: nav.launch world and added tsukinome

File: akatsuki_description/urdf/bot.xacro (robot description, xacro)
@@ -37,5 +37,5 @@
     </collision>
   </link>
-<link name="base_footprint">
+<!-- <link name="base_footprint">
 </link>
 <joint name="base_joint" type="fixed">
@@ -47,5 +47,5 @@
     <child
       link="obito_base" />
-</joint>
+</joint>     -->
  <link
     name="logo_link">
@@ -270,4 +270,5 @@
       xyz="1 0 0" />
   </joint>
+<!--
 <joint name="bot_cam_joint" type="fixed">
     <axis xyz="0 0 0" />
@@ -309,4 +310,5 @@
     <link name="camera_depth_frame">
   </link>
+ -->
 <link name="laser">
     <origin rpy="0 0 0" xyz="0 0 0"/>

Commit message: Major|update|added gfx plugin, navigation is working just fine

File: akatsuki_description/urdf/bot.xacro (robot description, xacro)
@@ -7,6 +7,6 @@
     <inertial>
       <origin
-   xyz="0 0.0 0"
-        rpy="0 0 3.142" />
+   xyz="0 0.0 0.12"
+        rpy="0 0 0" />
       <mass
         value="28" />
@@ -19,5 +19,5 @@
       <geometry>
         <mesh
-          filename="package://akatsuki_description/meshes/stl/only_chassis.stl" />
+          filename="package://akatsuki_description/meshes/stl/new_chassis.stl" />
       </geometry>
       <material
@@ -33,5 +33,5 @@
       <geometry>
      <mesh
-          filename="package://akatsuki_description/meshes/stl/only_chassis.stl" />
+          filename="package://akatsuki_description/meshes/stl/new_chassis.stl" />
       </geometry>
     </collision>
@@ -109,8 +109,8 @@
     <collision>
       <origin
-         xyz="0.05 0 0"
-        rpy="0 1.5707 0" />
-      <geometry>
-          <cylinder length="0.1" radius="0.12"/>
+         xyz="0 0.025 0"
+        rpy="1.5707 0 0" />
+      <geometry>
+          <cylinder length="0.05" radius="0.1"/>
       </geometry>
     </collision>
@@ -120,5 +120,5 @@
     type="continuous">
     <origin
-      xyz="0.27 -0.3 0"
+      xyz="0.2 0.2 0"
       rpy="0 0 0" />
     <parent
@@ -127,5 +127,5 @@
       link="front_wheel_left" />
     <axis
-      xyz="1 0 0" />
+      xyz="0 1 0" />
   </joint>
 <!-- rear wheel left -->
@@ -156,8 +156,8 @@
     <collision>
       <origin
-         xyz="0.05 0 0"
-        rpy="0 1.5707 0" />
-      <geometry>
-         <cylinder length="0.1" radius="0.12"/>
+         xyz="0 0.025  0"
+        rpy="1.5707 0 0" />
+      <geometry>
+         <cylinder length="0.05" radius="0.1"/>
       </geometry>
     </collision>
@@ -167,5 +167,5 @@
     type="continuous">
     <origin
-      xyz="0.27 0.3 0"
+      xyz="-0.2 0.2 0"
       rpy="0 0 0" />
     <parent
@@ -174,5 +174,5 @@
       link="rear_wheel_left" />
     <axis
-      xyz="1 0 0" />
+      xyz="0 1 0" />
   </joint>
 <!--   front wheel right -->
@@ -203,8 +203,8 @@
    <collision>
       <origin
-         xyz="-0.05 0 0"
-        rpy="0 1.5707 0" />
-      <geometry>
-          <cylinder length="0.1" radius="0.12"/>
+         xyz="0 -0.025 0"
+        rpy="1.5707 0 0" />
+      <geometry>
+          <cylinder length="0.05" radius="0.1"/>
       </geometry>
     </collision>
@@ -214,5 +214,5 @@
     type="continuous">
     <origin
-      xyz="-0.27 -0.3 0"
+      xyz="0.2 -0.2 0"
       rpy="0 0 0" />
     <parent
@@ -221,5 +221,5 @@
       link="front_wheel_right" />
     <axis
-      xyz="1 0 0" />
+      xyz="0 1 0" />
   </joint>
 <!--   rear wheel right -->
@@ -250,8 +250,8 @@
    <collision>
       <origin
-         xyz="-0.05 0 0"
-        rpy="0 1.5707 0" />
-      <geometry>
-          <cylinder length="0.1" radius="0.12"/>
+         xyz="0 -0.025 0"
+        rpy="1.5707 0 0" />
+      <geometry>
+          <cylinder length="0.05" radius="0.1"/>
       </geometry>
     </collision>
@@ -261,5 +261,5 @@
     type="continuous">
     <origin
-      xyz="-0.27 0.3 0"
+      xyz="-0.2 -0.2 0"
       rpy="0 0 0" />
     <parent
@@ -268,5 +268,5 @@
       link="rear_wheel_right" />
     <axis
-      xyz="1 0 0" />
+      xyz="0 1 0" />
   </joint>
 <!--
@@ -331,6 +331,5 @@
   </link>
   <joint name="lidar_joint" type="fixed">
-    <axis xyz="0 1 0"/>
-    <origin xyz="0 -0.36 0.23"
+    <origin xyz="0.26 0 0.15"
       rpy="0 0 -1.571" />
     <parent link="obito_base"/>
